File: FPS 100/Backplane/Backplane.kicad_pcb (KiCad board)
At the start: 6 copper layers, 384.7 x 240.4 mm, 27 parts

Commit message: 2026/1/9
Routing:
- net DPMBS16*: track 0.00 -> 446.0 mm, vias 0 -> 8
- net TM2A1: track 0.00 -> 244.4 mm, vias 0 -> 1
- net NOP*: track 0.00 -> 191.4 mm, vias 0 -> 1
- net MD01*: track 0.00 -> 185.8 mm, vias 0 -> 1
- net A1MBS14*: track 0.00 -> 154.1 mm, vias 0 -> 2
- net TM2DP: track 0.00 -> 136.0 mm, vias 0 -> 2
- net FMM16*: track 0.00 -> 131.1 mm, vias 0 -> 6
- net FMM18*: track 0.00 -> 129.5 mm, vias 0 -> 3
- net FMM19*: track 0.00 -> 129.2 mm, vias 0 -> 3
- net FMM17*: track 0.00 -> 127.6 mm, vias 0 -> 3
- net FAM17*: track 0.00 -> 121.6 mm, vias 0 -> 3
- net FAM16*: track 0.00 -> 118.7 mm, vias 0 -> 3
- net M1MBS23*: track 0.00 -> 113.9 mm, vias 0 -> 7
- net FAM18*: track 0.00 -> 107.1 mm, vias 0 -> 3
- net FAM19*: track 0.00 -> 102.9 mm, vias 0 -> 3
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
Commit message: 2026/1/10
Connections:
- net TST renamed TST0
- 4429_FMT_J1 pad 13: CTCLK -> CTLCLK
Routing:
- net PNL13*: track 0.00 -> 214.8 mm, vias 0 -> 5
- net PNL12*: track 0.00 -> 214.0 mm, vias 0 -> 4
- net PNL15*: track 0.00 -> 206.1 mm, vias 0 -> 5
- net DA13*: track 0.00 -> 205.7 mm, vias 0 -> 2
- net PNL14*: track 0.00 -> 205.0 mm, vias 0 -> 3
- net DA15*: track 0.00 -> 199.0 mm, vias 0 -> 3
- net DA14*: track 0.00 -> 189.5 mm, vias 0 -> 3
- net DA12*: track 0.00 -> 188.6 mm, vias 0 -> 3
- net FMM20*: track 0.00 -> 147.2 mm, vias 0 -> 3
- net FMM22*: track 0.00 -> 138.2 mm, vias 0 -> 4
- net FMM21*: track 0.00 -> 137.1 mm, vias 0 -> 3
- net A1MBS22*: track 0.00 -> 127.9 mm, vias 0 -> 4
- net A1MBS20*: track 0.00 -> 116.8 mm, vias 0 -> 2
- net A1MBS21*: track 0.00 -> 110.4 mm, vias 0 -> 3
- net FMM23*: track 0.00 -> 63.1 mm, vias 0 -> 2
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
Commit message: 2026/1/12
Parts:
- moved UNIBUS_XFER_J1 90.6 mm to (259.7, 420.1)
Routing:
- net DPMBS15*: track 0.00 -> 496.1 mm, vias 0 -> 9
- net DPMBS13*: track 0.00 -> 477.2 mm, vias 0 -> 10
- net DPMBS12*: track 0.00 -> 474.3 mm, vias 0 -> 8
- net DPMBS14*: track 0.00 -> 434.6 mm, vias 0 -> 7
- net MDI04: track 0.00 -> 362.4 mm, vias 0 -> 4
- net DPMBS10*: track 0.00 -> 360.1 mm, vias 0 -> 5
- net MDI06: track 0.00 -> 358.2 mm, vias 0 -> 4
- net DPMBS11*: track 0.00 -> 295.9 mm, vias 0 -> 9
- net DPEBS06*: track 0.00 -> 294.5 mm, vias 0 -> 6
- net DPEBS04*: track 0.00 -> 286.1 mm, vias 0 -> 6
- net DPEBS05*: track 0.00 -> 281.0 mm, vias 0 -> 7
- net !HRSET*: track 0.00 -> 278.9 mm, vias 0 -> 1
- net DPA2PNL*: track 0.00 -> 261.1 mm, vias 0 -> 4
- net DMA10*: track 0.00 -> 259.9 mm, vias 0 -> 3
- net +5V: track 2785.5 -> 3042.1 mm, vias 2 -> 4
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Other:
- board size 384.7 x 240.4 mm -> 397.9 x 240.4 mm

Commit message: 2026/1/13
Routing:
- net MDI07: track 0.00 -> 399.9 mm, vias 0 -> 5
- net MD05*: track 0.00 -> 390.0 mm, vias 0 -> 2
- net MD06*: track 0.00 -> 389.0 mm, vias 0 -> 2
- net MD07*: track 0.00 -> 386.6 mm, vias 0 -> 2
- net MD11*: track 0.00 -> 333.8 mm, vias 0 -> 8
- net MD09*: track 0.00 -> 328.2 mm, vias 0 -> 4
- net MD10*: track 0.00 -> 321.9 mm, vias 0 -> 6
- net MDI09: track 0.00 -> 319.9 mm, vias 0 -> 3
- net MDI10: track 0.00 -> 314.4 mm, vias 0 -> 5
- net MDI11: track 0.00 -> 313.9 mm, vias 0 -> 2
- net MDI08: track 0.00 -> 308.0 mm, vias 0 -> 4
- net SELREGB: track 0.00 -> 296.8 mm, vias 0 -> 2
- net MD04*: track 0.00 -> 295.8 mm, vias 0 -> 4
- net MD08*: track 0.00 -> 276.8 mm, vias 0 -> 7
- net PSZIP*: track 0.00 -> 261.2 mm, vias 0 -> 3
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
Commit message: 2026/1/13
Routing:
- net MD2DP: track 0.00 -> 234.0 mm, vias 0 -> 3
- net MD32*: track 0.00 -> 201.3 mm, vias 0 -> 11
- net 376IN*: track 0.00 -> 185.4 mm, vias 0 -> 2
- net 376LD*: track 0.00 -> 180.2 mm, vias 0 -> 4
- net PS1WRT: track 0.00 -> 140.9 mm, vias 0 -> 2
- net RTM*: track 0.00 -> 53.1 mm, vias 0 -> 1
- net FMM23*: track 63.1 -> 104.9 mm, vias 2 -> 3
- net PS0WRT: track 68.3 -> 66.3 mm
- net MDI36: track 180.0 -> 180.2 mm, vias 4 -> 5

Commit message: 2026/1/13
Routing:
- net A1EBS03*: track 47.0 -> 175.9 mm, vias 2 -> 7
- net TMNEG: track 0.00 -> 50.2 mm, vias 0 -> 2
