File: FPS 100/Backplane/Backplane.kicad_pcb (KiCad board)
At the start: 6 copper layers, 397.9 x 240.4 mm, 27 parts

Commit message: 2026/1/15
Connections:
- 4422_P1_J3 pad 90: LD0MA* -> LDOMA*
Routing:
- net +5V: track 3042.1 -> 6049.4 mm
- net A1EBS11*: track 0.00 -> 331.5 mm, vias 0 -> 3
- net A1EBS10*: track 0.00 -> 330.1 mm, vias 0 -> 3
- net A1EBS08*: track 0.00 -> 319.8 mm, vias 0 -> 3
- net DPEBS08*: track 0.00 -> 316.0 mm, vias 0 -> 5
- net A1EBS09*: track 0.00 -> 315.9 mm, vias 0 -> 3
- net DPEBS09*: track 0.00 -> 315.1 mm, vias 0 -> 6
- net A2EBS09*: track 0.00 -> 303.9 mm, vias 0 -> 2
- net A2EBS10*: track 0.00 -> 295.3 mm, vias 0 -> 2
- net DPEBS11*: track 0.00 -> 290.4 mm, vias 0 -> 5
- net A2EBS08*: track 0.00 -> 286.8 mm, vias 0 -> 3
- net A2EBS11*: track 0.00 -> 286.1 mm, vias 0 -> 2
- net DPEBS10*: track 0.00 -> 281.0 mm, vias 0 -> 5
- net WDPI: track 0.00 -> 271.8 mm, vias 0 -> 2
- net ABORT*: track 83.0 -> 352.9 mm, vias 1 -> 4
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
Commit message: 2026/1/18
Routing:
- net DPMBS01*: track 0.00 -> 379.4 mm, vias 0 -> 4
- net DPMBS02*: track 0.00 -> 374.2 mm, vias 0 -> 4
- net DPMBS05*: track 0.00 -> 362.3 mm, vias 0 -> 5
- net DPMBS06*: track 0.00 -> 362.1 mm, vias 0 -> 6
- net DPMBS04*: track 0.00 -> 361.6 mm, vias 0 -> 7
- net DPMBS07*: track 0.00 -> 358.5 mm, vias 0 -> 6
- net DPMBS03*: track 0.00 -> 350.6 mm, vias 0 -> 3
- net DPMBS00*: track 0.00 -> 327.0 mm, vias 0 -> 3
- net MDI17: track 0.00 -> 301.5 mm, vias 0 -> 3
- net MDI16: track 0.00 -> 295.8 mm, vias 0 -> 2
- net MDI15: track 0.00 -> 293.7 mm, vias 0 -> 2
- net MD17*: track 0.00 -> 287.5 mm, vias 0 -> 3
- net MD16*: track 0.00 -> 281.9 mm, vias 0 -> 2
- net MD14*: track 0.00 -> 279.3 mm, vias 0 -> 3
- net MD12*: track 0.00 -> 278.1 mm, vias 0 -> 3
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
Commit message: 2026/1/19
Routing:
- net DPMBS09*: track 0.00 -> 323.4 mm, vias 0 -> 6
- net DPMBS08*: track 0.00 -> 274.9 mm, vias 0 -> 5
- net Y2M2: track 15.8 -> 259.2 mm, vias 2 -> 6
- net DBLSW*: track 0.00 -> 238.6 mm, vias 0 -> 1
- net Y2A1: track 15.2 -> 242.7 mm, vias 2 -> 3
- net DP2M1: track 16.4 -> 242.7 mm, vias 2 -> 3
- net CB2A1E*: track 0.00 -> 225.1 mm, vias 0 -> 1
- net Y2M1: track 15.9 -> 239.2 mm, vias 2 -> 5
- net MD21*: track 0.00 -> 212.7 mm, vias 0 -> 3
- net MD23*: track 0.00 -> 212.7 mm, vias 0 -> 4
- net MD22*: track 0.00 -> 212.4 mm, vias 0 -> 4
- net MD20*: track 0.00 -> 204.4 mm, vias 0 -> 4
- net Y2A2: track 16.8 -> 213.5 mm, vias 0 -> 2
- net DP2A2M: track 17.8 -> 211.9 mm, vias 2 -> 3
- net MDI23: track 0.00 -> 190.8 mm, vias 0 -> 2
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
Commit message: 2026/1/19
Routing:
- net M1MBS02*: track 0.00 -> 317.2 mm, vias 0 -> 4
- net M1MBS03*: track 0.00 -> 230.5 mm, vias 0 -> 3
- net M1MBS01*: track 0.00 -> 228.0 mm, vias 0 -> 4
- net M1MBS00*: track 0.00 -> 226.9 mm, vias 0 -> 4
- net M2MBS03*: track 0.00 -> 210.5 mm, vias 0 -> 3
- net M2MBS01*: track 0.00 -> 210.4 mm, vias 0 -> 3
- net M2MBS02*: track 0.00 -> 210.1 mm, vias 0 -> 3
- net M2MBS00*: track 0.00 -> 209.8 mm, vias 0 -> 3
- net SP+DP04*: track 0.00 -> 161.7 mm, vias 0 -> 4
- net M1MBS04*: track 0.00 -> 156.4 mm, vias 0 -> 3
- net M1MBS05*: track 0.00 -> 153.2 mm, vias 0 -> 3
- net XIB: track 15.9 -> 142.7 mm, vias 2 -> 4
- net SP+DP12*: track 0.00 -> 123.0 mm, vias 0 -> 3
- net SP+DP14*: track 0.00 -> 121.1 mm, vias 0 -> 4
- net YLMCLKE*: track 16.2 -> 135.0 mm, vias 2 -> 3
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