File: FPS 100/Backplane_v2/Backplane_v2.kicad_pcb (KiCad board)
At the start: 6 copper layers, 397.9 x 240.4 mm, 67 parts, among them J1 Conn_01x02_Pin, J10 Conn_01x02_Pin, J11 Conn_01x02_Pin, J12 Conn_01x02_Pin, J13 Conn_01x02_Pin, J14 Conn_01x02_Pin, J15 Conn_01x02_Pin, J16 Conn_01x02_Pin, J17 Conn_01x02_Pin, J18 Conn_01x02_Pin, J19 Conn_01x02_Pin, J2 Conn_01x02_Pin, J20 Conn_01x02_Pin, J21 Conn_01x02_Pin, J22 Conn_01x02_Pin, J23 Conn_01x02_Pin, J24 Conn_01x02_Pin, J25 Conn_01x02_Pin, J26 Conn_01x02_Pin, J27 Conn_01x02_Pin, J28 Conn_01x02_Pin, J29 Conn_01x02_Pin, J3 Conn_01x02_Pin, J30 Conn_01x02_Pin, J31 Conn_01x02_Pin, J32 Conn_01x02_Pin, J33 Conn_01x02_Pin, J34 Conn_01x02_Pin, J35 Conn_01x02_Pin, J36 Conn_01x02_Pin, J37 Conn_01x02_Pin, J38 Conn_01x02_Pin, J39 Indicator Panel, J4 Conn_01x02_Pin, J6 Conn_01x02_Pin, J7 Conn_01x02_Pin, J8 Conn_01x02_Pin, J9 Conn_01x02_Pin

Commit message: 2026/1/20
Parts:
- added J40: Conn_01x02_Pin, User:TwistedPairHeader, F.Cu at (221.0, 488.3)
- added J41: Conn_01x02_Pin, User:TwistedPairHeader, F.Cu at (542.9, 446.5)
- moved J38 14.0 mm to (292.1, 446.4)
Connections:
- 4408_P3_J2 pad 115: EXTCLK{408} -> Net-(J40-Pin_2)
- 4421_PDP_IF_J1 pad 6: unconnected-(4421_PDP_IF_J1-Pad6) -> Net-(J41-Pin_2)
Routing:
- net Net-(J38-Pin_2): track 10.8 -> 4.44 mm
- net Net-(J41-Pin_2): track 0.00 -> 4.84 mm
- net Net-(J40-Pin_2): track 0.00 -> 4.44 mm
- net +5V: track 6048.4 -> 6052.3 mm, vias 36 -> 102
- net DPMBS18*: track 405.4 -> 403.6 mm
- net DPMBS17*: track 404.7 -> 406.0 mm
- net BUF2CLK: track 90.5 -> 91.7 mm
- net INTOP: track 70.2 -> 69.1 mm
- net I+H13: track 296.7 -> 297.8 mm
- net BH2HD: track 321.2 -> 322.2 mm
- net DPMBS20*: track 411.3 -> 412.3 mm
- net HD10: track 163.3 -> 164.4 mm
- net BL2HD: track 208.9 -> 210.0 mm
- net SR2HD*: track 290.5 -> 291.5 mm
- net DPMBS19*: track 456.7 -> 455.9 mm
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
Commit message: 2026/1/21
Parts:
- moved UNIBUS_XFER_J2 70.4 mm to (396.2, 429.3)
- moved UNIBUS_XFER_J1 43.5 mm to (302.3, 429.3)
- moved J39 23.3 mm to (487.7, 429.3)
- moved J1 15.7 mm to (535.9, 600.1), turned to 90 degrees
- moved J2 14.6 mm to (530.9, 600.1)
- moved J3 14.6 mm to (525.8, 600.1)
Routing:
- net +5V: track 6052.3 -> 3090.4 mm
- net BUSINIT*: track 0.00 -> 176.6 mm
- net BUSSSYN*: track 0.00 -> 172.8 mm, vias 0 -> 1
- net BUSC01*: track 0.00 -> 163.8 mm, vias 0 -> 1
- net DMAIND: track 0.00 -> 158.8 mm
- net RUNIND: track 0.00 -> 155.1 mm
- net BUSNPR*: track 0.00 -> 144.9 mm
- net BUSD01*: track 0.00 -> 137.5 mm, vias 0 -> 1
- net BUSD00*: track 0.00 -> 137.0 mm, vias 0 -> 1
- net BUSSACK*: track 0.00 -> 136.1 mm
- net BUSA17*: track 0.00 -> 133.5 mm, vias 0 -> 1
- net BUSD02*: track 0.00 -> 133.3 mm, vias 0 -> 1
- net BUSNPGOUT: track 0.00 -> 131.1 mm
- net BUSD03*: track 0.00 -> 130.0 mm, vias 0 -> 1
- net BUSBGOUT: track 0.00 -> 119.3 mm, vias 0 -> 1
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Other:
- board size 397.9 x 240.4 mm -> 440 x 205 mm
