File: FPS 100/Backplane_v2/Backplane_v2.kicad_sch (KiCad schematic)
At the start: 27 parts

Commit message: 2026/1/20
Parts:
- added J1, J10, J11, J12, J13, J14, J15, J16, J17, J18, J19, J2, J20, J21, J22, J23, J24, J25, J26, J27, J28, J29, J3, J30, J31, J32, J33, J34, J35, J36, J37, J38, J4, J6, J7, J8, J9: Conn_01x02_Pin, User:TwistedPairHeader, symbol Connector:Conn_01x02_Pin
- added J39: Indicator Panel, Connector_PinHeader_2.54mm:PinHeader_1x04_P2.54mm_Vertical, symbol Connector:Conn_01x04_Pin
- added J5: ~, User:TwistedPairHeader, symbol Connector:Conn_01x02_Pin
- added UNIBUS_XFER_J2: Conn_02x25_Odd_Even, Connector_PinHeader_2.54mm:PinHeader_2x25_P2.54mm_Vertical, symbol Connector_Generic:Conn_02x25_Odd_Even
Connections:
- net BUSBGOUT: now also UNIBUS_XFER_J2.49 (Pin_49); no longer UNIBUS_XFER_J1.50 (Pin_50)
- net BUSC01*: now also UNIBUS_XFER_J2.37 (Pin_37); no longer UNIBUS_XFER_J1.38 (Pin_38)
- net BUSD00*: now also UNIBUS_XFER_J2.1 (Pin_1); no longer UNIBUS_XFER_J1.2 (Pin_2)
- net BUSD01*: now also UNIBUS_XFER_J2.3 (Pin_3); no longer UNIBUS_XFER_J1.4 (Pin_4)
- net BUSD02*: now also UNIBUS_XFER_J2.5 (Pin_5); no longer UNIBUS_XFER_J1.6 (Pin_6)
- net BUSD03*: now also UNIBUS_XFER_J2.7 (Pin_7); no longer UNIBUS_XFER_J1.8 (Pin_8)
- net BUSD04*: now also UNIBUS_XFER_J2.9 (Pin_9); no longer UNIBUS_XFER_J1.10 (Pin_10)
- net BUSD05*: now also UNIBUS_XFER_J2.11 (Pin_11); no longer UNIBUS_XFER_J1.12 (Pin_12)
- net BUSD06*: now also UNIBUS_XFER_J2.13 (Pin_13); no longer UNIBUS_XFER_J1.14 (Pin_14)
- net BUSD07*: now also UNIBUS_XFER_J2.15 (Pin_15); no longer UNIBUS_XFER_J1.16 (Pin_16)
- net BUSD08*: now also UNIBUS_XFER_J2.17 (Pin_17); no longer UNIBUS_XFER_J1.18 (Pin_18)
- net BUSD09*: now also UNIBUS_XFER_J2.19 (Pin_19); no longer UNIBUS_XFER_J1.20 (Pin_20)
- net BUSD10*: now also UNIBUS_XFER_J2.21 (Pin_21); no longer UNIBUS_XFER_J1.22 (Pin_22)
- net BUSD11*: now also UNIBUS_XFER_J2.23 (Pin_23); no longer UNIBUS_XFER_J1.24 (Pin_24)
- net BUSD12*: now also UNIBUS_XFER_J2.25 (Pin_25); no longer UNIBUS_XFER_J1.26 (Pin_26)
- net BUSD13*: now also UNIBUS_XFER_J2.27 (Pin_27); no longer UNIBUS_XFER_J1.28 (Pin_28)
- net BUSD14*: now also UNIBUS_XFER_J2.29 (Pin_29); no longer UNIBUS_XFER_J1.30 (Pin_30)
- net BUSD15*: now also UNIBUS_XFER_J2.31 (Pin_31); no longer UNIBUS_XFER_J1.32 (Pin_32)
- net BUSINIT*: now also UNIBUS_XFER_J2.43 (Pin_43); no longer UNIBUS_XFER_J1.44 (Pin_44)
- net BUSNPGOUT: now also UNIBUS_XFER_J2.47 (Pin_47); no longer UNIBUS_XFER_J1.48 (Pin_48)
- net BUSNPR*: now also UNIBUS_XFER_J2.41 (Pin_41); no longer UNIBUS_XFER_J1.42 (Pin_42)
- net BUSSACK*: now also UNIBUS_XFER_J2.39 (Pin_39); no longer UNIBUS_XFER_J1.40 (Pin_40)
- net BUSSSYN*: now also UNIBUS_XFER_J2.45 (Pin_45); no longer UNIBUS_XFER_J1.46 (Pin_46)
- net DMAIND: now also J39.3 (Pin_3)
- net GND: now also UNIBUS_XFER_J1.10 (Pin_10), UNIBUS_XFER_J1.12 (Pin_12), UNIBUS_XFER_J1.14 (Pin_14), UNIBUS_XFER_J1.16 (Pin_16), UNIBUS_XFER_J1.18 (Pin_18), UNIBUS_XFER_J1.2 (Pin_2), UNIBUS_XFER_J1.20 (Pin_20), UNIBUS_XFER_J1.22 (Pin_22), UNIBUS_XFER_J1.24 (Pin_24), UNIBUS_XFER_J1.26 (Pin_26), UNIBUS_XFER_J1.28 (Pin_28), UNIBUS_XFER_J1.30 (Pin_30), UNIBUS_XFER_J1.32 (Pin_32), UNIBUS_XFER_J1.34 (Pin_34), UNIBUS_XFER_J1.36 (Pin_36), UNIBUS_XFER_J1.38 (Pin_38), UNIBUS_XFER_J1.4 (Pin_4), UNIBUS_XFER_J1.40 (Pin_40), UNIBUS_XFER_J1.42 (Pin_42), UNIBUS_XFER_J1.44 (Pin_44), UNIBUS_XFER_J1.46 (Pin_46), UNIBUS_XFER_J1.48 (Pin_48), UNIBUS_XFER_J1.50 (Pin_50), UNIBUS_XFER_J1.6 (Pin_6), UNIBUS_XFER_J1.8 (Pin_8), J1.1 (Pin_1), J10.1 (Pin_1), J11.1 (Pin_1), J12.2 (Pin_2), J13.1 (Pin_1), J14.2 (Pin_2), J15.2 (Pin_2), J16.1 (Pin_1), J17.2 (Pin_2), J18.2 (Pin_2), J19.1 (Pin_1), J2.1 (Pin_1), J20.2 (Pin_2), J21.2 (Pin_2), J22.2 (Pin_2), J23.2 (Pin_2), J24.2 (Pin_2), J25.1 (Pin_1), J26.1 (Pin_1), J27.1 (Pin_1), J28.1 (Pin_1), J29.1 (Pin_1), J3.1 (Pin_1), J30.1 (Pin_1), J31.1 (Pin_1), J32.1 (Pin_1), J33.1 (Pin_1), J34.1 (Pin_1), J35.2 (Pin_2), J36.2 (Pin_2), J37.2 (Pin_2), J38.1 (Pin_1), J4.2 (Pin_2), J5.1 (Pin_1), J6.2 (Pin_2), J7.1 (Pin_1), J8.2 (Pin_2), J9.1 (Pin_1), UNIBUS_XFER_J2.10 (Pin_10), UNIBUS_XFER_J2.12 (Pin_12), UNIBUS_XFER_J2.14 (Pin_14), UNIBUS_XFER_J2.16 (Pin_16), UNIBUS_XFER_J2.18 (Pin_18), UNIBUS_XFER_J2.2 (Pin_2), UNIBUS_XFER_J2.20 (Pin_20), UNIBUS_XFER_J2.22 (Pin_22), UNIBUS_XFER_J2.24 (Pin_24), UNIBUS_XFER_J2.26 (Pin_26), UNIBUS_XFER_J2.28 (Pin_28), UNIBUS_XFER_J2.30 (Pin_30), UNIBUS_XFER_J2.32 (Pin_32), UNIBUS_XFER_J2.34 (Pin_34), UNIBUS_XFER_J2.36 (Pin_36), UNIBUS_XFER_J2.38 (Pin_38), UNIBUS_XFER_J2.4 (Pin_4), UNIBUS_XFER_J2.40 (Pin_40), UNIBUS_XFER_J2.42 (Pin_42), UNIBUS_XFER_J2.44 (Pin_44), UNIBUS_XFER_J2.46 (Pin_46), UNIBUS_XFER_J2.48 (Pin_48), UNIBUS_XFER_J2.50 (Pin_50), UNIBUS_XFER_J2.6 (Pin_6), UNIBUS_XFER_J2.8 (Pin_8)
- net HINTIND: now also J39.2 (Pin_2)
- net INTIND: now also J39.1 (Pin_1)
- net RUNIND: now also J39.4 (Pin_4)
- removed net !A1CLK: 4401_FA_J1.8, 4408_P3_J1.15, 4426_FM_J1.8
- removed net !A2CLK: 4401_FA_J1.10, 4408_P3_J1.14, 4426_FM_J1.10
- net !CBCLK1: no longer names the net of 4422_P1_J3.7
- net !CBCLK1: now also J18.1 (Pin_1); no longer 4408_P3_J1.8
- net !CBCLK2: no longer names the net of 4408_P3_J1.7
- net !CBCLK2: now also J21.1 (Pin_1); no longer 4423_P2_J1.5
- net !DPLCLK: no longer names the net of 4402_DPL_J1.5
- net !DPLCLK: now also J4.1 (Pin_1); no longer 4408_P3_J1.16
- net !DPRCLK: no longer names the net of 4408_P3_J1.17
- net !DPRCLK: now also J28.2 (Pin_2); no longer 4402_DPR_J1.5
- net !FACLK: no longer names the net of 4408_P3_J1.19
- net !FACLK: now also J27.2 (Pin_2); no longer 4401_FA_J1.6
- net !FMCLK: no longer names the net of 4426_FM_J1.6
- net !FMCLK: now also J9.2 (Pin_2); no longer 4408_P3_J1.13
- net !HRSET*: no longer names the net of 4421_PDP_IF_J2.52
- net !HRSET*: now also J38.2 (Pin_2); no longer 4408_P3_J1.25
- net !IOCLK: no longer names the net of 4408_P3_J1.20
- net !IOCLK: now also J35.1 (Pin_1)
- net !MCLK: no longer names the net of 4408_P3_J1.21
- net !MCLK: now also J26.2 (Pin_2); no longer 4424_MD_J1.5
- net !MICLK: no longer names the net of 4426_FM_J1.5
- net !MICLK: now also J8.1 (Pin_1); no longer 4408_P3_J1.12
- net !SPCLK: no longer names the net of 4422_P1_J3.6
- net !SPCLK: now also J19.2 (Pin_2); no longer 4408_P3_J1.5
- net !T75: no longer names the net of 4408_P3_J1.11
- net !T75: now also J23.1 (Pin_1); no longer 4424_MD_J1.6
- net !TMCLK: no longer names the net of 4408_P3_J1.10
- net !TMCLK: now also J32.2 (Pin_2); no longer 4425_TM_J1.5
- removed net !WRT*: 4408_P3_J1.6, 4422_P1_J3.5, 4423_P2_J1.6
- net !WRTL*: no longer names the net of 4402_DPL_J1.6
- net !WRTL*: now also J5.2 (Pin_2); no longer 4408_P3_J1.18
- net !WRTR*: no longer names the net of 4408_P3_J1.9
- net !WRTR*: now also J22.1 (Pin_1); no longer 4402_DPR_J1.6
- new net: 4422_P1_J3.5, J17.1 (Pin_1)
- new net: 4426_FM_J1.10, J11.2 (Pin_2)
- new net: 4426_FM_J1.8, J10.2 (Pin_2)
- new net: 4408_P3_J1.5, J20.1 (Pin_1)
- new net: 4408_P3_J1.15, J29.2 (Pin_2)
- new net: 4408_P3_J1.12, J33.2 (Pin_2)
- new net: 4408_P3_J1.13, J24.1 (Pin_1)
- new net: 4408_P3_J1.14, J34.2 (Pin_2)
- new net: 4408_P3_J1.16, J37.1 (Pin_1)
- new net: 4408_P3_J1.18, J36.1 (Pin_1)
- new net: 4408_P3_J1.25, J25.2 (Pin_2)
- new net: 4408_P3_J1.6, J30.2 (Pin_2)
- new net: 4408_P3_J1.8, J31.2 (Pin_2)
- new net: 4401_FA_J1.10, J3.2 (Pin_2)
- new net: 4424_MD_J1.5, J12.1 (Pin_1)
- new net: 4424_MD_J1.6, J13.2 (Pin_2)
- new net: 4401_FA_J1.6, J1.2 (Pin_2)
- new net: 4401_FA_J1.8, J2.2 (Pin_2)
- new net: 4423_P2_J1.5, J15.1 (Pin_1)
- new net: 4423_P2_J1.6, J16.2 (Pin_2)
- new net: 4402_DPR_J1.5, J6.1 (Pin_1)
- new net: 4402_DPR_J1.6, J7.2 (Pin_2)
- new net: 4425_TM_J1.5, J14.1 (Pin_1)
Other:
- note added: "!SPCLK P3.A.005 <-> P1.A.006 !WRT* P3.A.006 <-> P1.A.005 <-> P2.A.006 !CBCLK2 P3.A.007 <-> P2.A.005 !CBCLK1 P3.A.008 <-> P1.A.007 !WRTR* P3.A.009 <-> DPR.A.006 !TMCLK P3.A.010 <-> TM.A.005 !T75 P3.A.011 <-> MD.A.006 !MICLK P3.A.012 <-> FM.A.005 !FMCLK P3.A.013 <-> FM.A.006 !A2CLK P3.A.014 <-> FA.A.010 <-> FM.A.010 !A1CLK P3.A.015 <-> FA.A.008 <-> FM.A.008 !DPLCLK P3.A.016 <-> DPL.A.005 !DPRCLK P3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"
- note added: "INDICATORS"
- moved on the sheet: UNIBUS_XFER_J1

Commit message: 2026/1/20
Parts:
- added J40, J41: Conn_01x02_Pin, User:TwistedPairHeader, symbol Connector:Conn_01x02_Pin
Connections:
- net GND: now also J40.1 (Pin_1), J41.1 (Pin_1)
- net at 4421_PDP_IF_J1.6: now also J41.2 (Pin_2)
- net EXTCLK{408}: no longer names the net of 4408_P3_J2.115
- net EXTCLK{408}: now also J40.2 (Pin_2)
Other:
- moved on the sheet: UNIBUS_XFER_J2

Commit message: 2026/1/21
Other:
- note added: "These are NOT etched Use external twisted pair wires !SPCLK P3.A.005 <-> P1.A.006 !WRT* P3.A.006 <-> P1.A.005 <-> P2.A.006 !CBCLK2 P3.A.007 <-> P2.A.005 !CBCLK1 P3.A.008 <-> P1.A.007 !WRTR* P3.A.009 <-> DPR.A.006 !TMCLK P3.A.010 <-> TM.A.005 !T75 P3.A.011 <-> MD.A.006 !MICLK P3.A.012 <-> FM.A.005 !FMCLK P3.A.013 <-> FM.A.006 !A2CLK P3.A.014 <-> FA.A.010 <-> FM.A.010 !A1CLK P3.A.015 <-> FA.A.008 <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"
- note removed: "!SPCLK P3.A.005 <-> P1.A.006 !WRT* P3.A.006 <-> P1.A.005 <-> P2.A.006 !CBCLK2 P3.A.007 <-> P2.A.005 !CBCLK1 P3.A.008 <-> P1.A.007 !WRTR* P3.A.009 <-> DPR.A.006 !TMCLK P3.A.010 <-> TM.A.005 !T75 P3.A.011 <-> MD.A.006 !MICLK P3.A.012 <-> FM.A.005 !FMCLK P3.A.013 <-> FM.A.006 !A2CLK P3.A.014 <-> FA.A.010 <-> FM.A.010 !A1CLK P3.A.015 <-> FA.A.008 <-> FM.A.008 !DPLCLK P3.A.016 <-> DPL.A.005 !DPRCLK P3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"
Changed lines of the file:
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@@
 		)
 	)
-	(text "!SPCLK      P3.A.005 <->  P1.A.006\n!WRT*       P3.A.006 <->  P1.A.005 <-> P2.A.006\n!CBCLK2     P3.A.007 <->  P2.A.005\n!CBCLK1     P3.A.008 <->  P1.A.007\n!WRTR*      P3.A.009 <-> DPR.A.006\n!TMCLK      P3.A.010 <->  TM.A.005\n!T75        P3.A.011 <->  MD.A.006\n!MICLK      P3.A.012 <->  FM.A.005\n!FMCLK      P3.A.013 <->  FM.A.006\n!A2CLK      P3.A.014 <->  FA.A.010 <-> FM.A.010\n!A1CLK      P3.A.015 <->  FA.A.008 <-> FM.A.008\n!DPLCLK     P3.A.016 <-> DPL.A.005\n!DPRCLK     P3.A.017 <-> DPR.A.005\n!WRTL*      P3.A.018 <-> DPL.A.006\n!FACLK      P3.A.019 <->  FA.A.006\n!IOCLK      P3.A.020 <->  IF.A.006\n!MCLK       P3.A.021 <->  MD.A.005\n!HRSET*     P3.A.025 <->  IF.B.052\nEXTCLK{408} P3.B.115 <-> External Clock (if jumpered)"
+	(text "These are NOT etched\nUse external twisted pair wires\n\n!SPCLK      P3.A.005 <->  P1.A.006\n!WRT*       P3.A.006 <->  P1.A.005 <-> P2.A.006\n!CBCLK2     P3.A.007 <->  P2.A.005\n!CBCLK1     P3.A.008 <->  P1.A.007\n!WRTR*      P3.A.009 <-> DPR.A.006\n!TMCLK      P3.A.010 <->  TM.A.005\n!T75        P3.A.011 <->  MD.A.006\n!MICLK      P3.A.012 <->  FM.A.005\n!FMCLK      P3.A.013 <->  FM.A.006\n!A2CLK      P3.A.014 <->  FA.A.010 <-> FM.A.010\n!A1CLK      P3.A.015 <->  FA.A.008 <-> FM.A.008\n!DPLCLK     P3.A.016 <-> DPL.A.005\n!DPRCLK     P3.A.017 <-> DPR.A.005\n!WRTL*      P3.A.018 <-> DPL.A.006\n!FACLK      P3.A.019 <->  FA.A.006\n!IOCLK      P3.A.020 <->  IF.A.006\n!MCLK       P3.A.021 <->  MD.A.005\n!HRSET*     P3.A.025 <->  IF.B.052\nEXTCLK{408} P3.B.115 <-> External Clock (if jumpered)"
 		(exclude_from_sim no)
-		(at 708.914 444.246 0)
+		(at 707.898 460.502 0)
 		(effects
 			(font
@@
 	(wire
 		(pts
+			(xy 664.21 367.03) (xy 643.89 367.03)
+		)
+		(stroke
+			(width 0)
+			(type default)
+		)
+	)
+	(wire
+		(pts
 			(xy 963.93 455.93) (xy 963.93 458.47)
 		)
@@
 	(wire
 		(pts
+			(xy 523.24 90.17) (xy 549.91 90.17)
+		)
+		(stroke
+			(width 0)
+			(type default)
+		)
+	)
+	(wire
+		(pts
 			(xy 923.29 420.37) (xy 923.29 422.91)
 		)
@@
 	(global_label "RBUEQ*"
 		(shape input)
-		(at 643.89 367.03 0)
+		(at 664.21 367.03 0)
 		(fields_autoplaced yes)
 		(effects
@@
 		)
 		(property "Intersheetrefs" "${INTERSHEET_REFS}"
-			(at 654.1928 367.03 0)
+			(at 674.5128 367.03 0)
 			(effects
 				(font
@@
 	(global_label "RBUFQ"
 		(shape input)
-		(at 549.91 90.17 180)
+		(at 523.24 90.17 180)
 		(fields_autoplaced yes)
 		(effects
@@
 		)
 		(property "Intersheetrefs" "${INTERSHEET_REFS}"
-			(at 540.6352 90.17 0)
+			(at 513.9652 90.17 0)
 			(effects
 				(font

Commit message: 2026/1/26
Connections:
- net DPALD*A is gone; now on net DPALD*: 4422_P1_J4.38
- net EXTNT is gone; now on net EXINT: 4408_P3_J2.100
- net PN2DBL* is gone; now on net PNL2DBL*: 4422_P1_J4.81
- net RBUFQ is gone; now on net RBUEQ*: 4423_P2_J1.23
Changed lines of the file:
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@@
 	(wire
 		(pts
-			(xy 664.21 367.03) (xy 643.89 367.03)
-		)
-		(stroke
-			(width 0)
-			(type default)
-		)
-	)
-	(wire
-		(pts
 			(xy 963.93 455.93) (xy 963.93 458.47)
 		)
@@
 	(wire
 		(pts
-			(xy 523.24 90.17) (xy 549.91 90.17)
-		)
-		(stroke
-			(width 0)
-			(type default)
-		)
-	)
-	(wire
-		(pts
 			(xy 923.29 420.37) (xy 923.29 422.91)
 		)
@@
 	(global_label "RBUEQ*"
 		(shape input)
-		(at 664.21 367.03 0)
+		(at 643.89 367.03 0)
 		(fields_autoplaced yes)
 		(effects
@@
 		)
 		(property "Intersheetrefs" "${INTERSHEET_REFS}"
-			(at 674.5128 367.03 0)
+			(at 654.1928 367.03 0)
 			(effects
 				(font
@@
 		)
 	)
-	(global_label "PN2DBL*"
+	(global_label "PNL2DBL*"
 		(shape input)
 		(at 631.19 323.85 180)
@@
 		)
 		(property "Intersheetrefs" "${INTERSHEET_REFS}"
-			(at 619.8591 323.85 0)
+			(at 618.831 323.85 0)
 			(effects
 				(font
@@
 		)
 	)
-	(global_label "RBUFQ"
+	(global_label "RBUEQ*"
 		(shape input)
-		(at 523.24 90.17 180)
+		(at 549.91 90.17 180)
 		(fields_autoplaced yes)
 		(effects
@@
 		)
 		(property "Intersheetrefs" "${INTERSHEET_REFS}"
-			(at 513.9652 90.17 0)
+			(at 539.6072 90.17 0)
 			(effects
 				(font
@@
 		)
 	)
-	(global_label "DPALD*A"
+	(global_label "DPALD*"
 		(shape input)
 		(at 643.89 267.97 0)
@@
 		)
 		(property "Intersheetrefs" "${INTERSHEET_REFS}"
-			(at 654.8581 267.97 0)
+			(at 653.7695 267.97 0)
 			(effects
 				(font
@@
 		)
 	)
-	(global_label "EXTNT"
+	(global_label "EXINT"
 		(shape input)
 		(at 720.09 346.71 0)
@@
 		)
 		(property "Intersheetrefs" "${INTERSHEET_REFS}"
-			(at 728.6994 346.71 0)
+			(at 728.3366 346.71 0)
 			(effects
 				(font
